File: Homework_2/Homework2.brd (EAGLE design)
At the start: 50 x 50 mm, 22 parts

Commit message: Homework2/3_commit4
more schematic work
Parts:
- moved U$2 81.4 mm to (40.6, 10.2), turned to 270 degrees
- moved U$4 79.1 mm to (16.5, 48.3)
- moved PICKIT 77.5 mm to (48.3, 48.3), turned to 270 degrees
- moved USER 45.0 mm to (2.54, 1.27)
- moved RESET 43.4 mm to (2.54, 6.35)
- moved 10UF_1 34.3 mm to (36.8, 19.1)
- moved 0.1UF_2 25.3 mm to (33.0, 38.1), turned to 270 degrees
Connections:
- removed net N$3: 8MHZRES.2
- new net N$10: 10UF_1.1, U$1.20
- new net N$8: 0.1UF_2.2, PICKIT.3, U$1.27
- new net N$9: 0.1UF_2.1, PICKIT.2, U$1.28
- net GND: now also 10UF_1.2, 8MHZRES.2, U$1.19
- net N$6: now also PICKIT.4; no longer PICKIT.3
- net N$7: now also PICKIT.5; no longer PICKIT.4
Changed lines of the file:
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@@
 <attribute name="PROD_ID" value="CONN-08438" x="1.27" y="16.51" size="1.778" layer="27" rot="R90" display="off"/>
 </element>
-<element name="PICKIT" library="Homework2" package="1X05" value="" x="-25.4" y="24.13"/>
+<element name="PICKIT" library="Homework2" package="1X05" value="" x="48.26" y="48.26" rot="R270"/>
 <element name="RED_LED" library="Homework2" package="LED3MM" value="" x="-20.32" y="31.75"/>
 <element name="GREEN_LED" library="Homework2" package="LED3MM" value="" x="-30.48" y="31.75"/>
 <element name="U$1" library="Homework2" package="DIL28-3" value="PIC32" x="25.4" y="22.86" rot="R270"/>
-<element name="U$2" library="Homework2" package="TO92" value="MCP1702" x="-39.37" y="25.4"/>
+<element name="U$2" library="Homework2" package="TO92" value="MCP1702" x="40.64" y="10.16" rot="R270"/>
 <element name="U$3" library="Homework2" package="USB-MB-H" value="USB_B_PCB" x="3.81" y="44.45"/>
-<element name="10UF_1" library="Homework2" package="C050-024X044" value="" x="58.42" y="45.72"/>
+<element name="10UF_1" library="Homework2" package="C050-024X044" value="" x="36.83" y="19.05"/>
 <element name="0.1UF_4" library="Homework2" package="C025-024X044" value="" x="57.15" y="40.64"/>
 <element name="0.1UF_1" library="Homework2" package="C025-024X044" value="" x="57.15" y="35.56"/>
-<element name="0.1UF_2" library="Homework2" package="C025-024X044" value="" x="57.15" y="30.48"/>
+<element name="0.1UF_2" library="Homework2" package="C025-024X044" value="" x="33.02" y="38.1" rot="R270"/>
 <element name="0.1UF_3" library="Homework2" package="C025-024X044" value="" x="57.15" y="25.4"/>
 <element name="330_R1" library="Homework2" package="0204/5" value="" x="58.42" y="21.59"/>
@@
 <element name="8MHZRES" library="SparkFun-FreqCtrl" package="RESONATOR-PTH" value="" x="15.24" y="17.78" rot="R90"/>
 <element name="10UF_2" library="Homework2" package="C050-024X044" value="" x="58.42" y="0"/>
-<element name="RESET" library="Homework2" package="1X03" value="" x="-39.37" y="-5.08"/>
-<element name="U$4" library="Homework2" package="SLIDER_FOOTPRINT" value="SLIDER_SWITCH" x="-36.83" y="-10.16"/>
-<element name="USER" library="Homework2" package="1X03" value="" x="-39.37" y="-15.24"/>
+<element name="RESET" library="Homework2" package="1X03" value="" x="2.54" y="6.35"/>
+<element name="U$4" library="Homework2" package="SLIDER_FOOTPRINT" value="SLIDER_SWITCH" x="16.51" y="48.26"/>
+<element name="USER" library="Homework2" package="1X03" value="" x="2.54" y="1.27"/>
 </elements>
 <signals>
@@
 <wire x1="15.24" y1="15.24" x2="21.59" y2="16.51" width="0" layer="19" extent="1-1"/>
 </signal>
-<signal name="N$3">
-<contactref element="8MHZRES" pad="2"/>
-</signal>
 <signal name="GND">
 <contactref element="U$2" pad="1"/>
+<contactref element="U$1" pad="19"/>
+<contactref element="10UF_1" pad="2"/>
+<contactref element="8MHZRES" pad="2"/>
+<wire x1="40.64" y1="11.43" x2="39.37" y2="19.05" width="0" layer="19" extent="1-1"/>
+<wire x1="29.21" y1="16.51" x2="39.37" y2="19.05" width="0" layer="19" extent="1-1"/>
+<wire x1="15.24" y1="17.78" x2="29.21" y2="16.51" width="0" layer="19" extent="1-1"/>
 </signal>
 <signal name="N$4">
@@
 <contactref element="PICKIT" pad="1"/>
 <contactref element="U$1" pad="1"/>
-<wire x1="-25.4" y1="24.13" x2="21.59" y2="39.37" width="0" layer="19" extent="1-1"/>
+<wire x1="48.26" y1="48.26" x2="21.59" y2="39.37" width="0" layer="19" extent="1-1"/>
+</signal>
+<signal name="N$8">
+<contactref element="0.1UF_2" pad="2"/>
+<contactref element="U$1" pad="27"/>
+<contactref element="PICKIT" pad="3"/>
+<wire x1="29.21" y1="36.83" x2="33.02" y2="36.83" width="0" layer="19" extent="1-1"/>
+<wire x1="48.26" y1="43.18" x2="29.21" y2="36.83" width="0" layer="19" extent="1-1"/>
+</signal>
+<signal name="N$9">
+<contactref element="0.1UF_2" pad="1"/>
+<contactref element="U$1" pad="28"/>
+<contactref element="PICKIT" pad="2"/>
+<wire x1="29.21" y1="39.37" x2="33.02" y2="39.37" width="0" layer="19" extent="1-1"/>
+<wire x1="48.26" y1="45.72" x2="29.21" y2="39.37" width="0" layer="19" extent="1-1"/>
 </signal>
 <signal name="N$6">
-<contactref element="PICKIT" pad="3"/>
+<contactref element="PICKIT" pad="4"/>
 <contactref element="U$1" pad="4"/>
-<wire x1="-20.32" y1="24.13" x2="21.59" y2="31.75" width="0" layer="19" extent="1-1"/>
+<wire x1="48.26" y1="40.64" x2="21.59" y2="31.75" width="0" layer="19" extent="1-1"/>
 </signal>
 <signal name="N$7">
-<contactref element="PICKIT" pad="4"/>
+<contactref element="PICKIT" pad="5"/>
 <contactref element="U$1" pad="5"/>
-<wire x1="-17.78" y1="24.13" x2="21.59" y2="29.21" width="0" layer="19" extent="1-1"/>
+<wire x1="48.26" y1="38.1" x2="21.59" y2="29.21" width="0" layer="19" extent="1-1"/>
+</signal>
+<signal name="N$10">
+<contactref element="U$1" pad="20"/>
+<contactref element="10UF_1" pad="1"/>
+<wire x1="29.21" y1="19.05" x2="34.29" y2="19.05" width="0" layer="19" extent="1-1"/>
 </signal>
 </signals>

Commit message: Homework_2/3_commit#5
finished schematic
Parts:
- moved RESET 55.8 mm to (39.4, 48.3)
- moved 330_R2 54.6 mm to (5.08, 6.35), turned to 180 degrees
- moved RED_LED 49.0 mm to (19.1, 2.54)
- moved GREEN_LED 38.8 mm to (2.54, 11.4)
- moved 330_R1 37.7 mm to (26.7, 1.27)
- moved 0.1UF_1 25.0 mm to (35.6, 48.3), turned to 180 degrees
- moved 10UF_2 15.3 mm to (47.0, 10.2), turned to 90 degrees
- moved U$2 4.02 mm to (36.8, 8.89)
Connections:
- net N$6 renamed PGED1
- net N$7 renamed PGEC1
- removed net N$4: U$3.GND
- removed net N$5: PICKIT.1, U$1.1
- new net +3V3: 10K_R3.2, 10K_R4.1
- new net A0: J2.8, U$1.2
- new net A1: J2.7, U$1.3
- new net A4: GREEN_LED.A, J2.3, U$1.12
- new net B13: J1.6, U$1.24
- new net B14: J1.7, U$1.25
- new net B15: J1.8, U$1.26
- new net B2: J2.6, U$1.6
- new net B3: J2.5, U$1.7
- new net B4: 10K_R4.2, J2.4, U$1.11, USER.3
- new net B7: J1.3, U$1.16
- new net B8: J1.4, U$1.17
- new net B9: J1.5, U$1.18
- new net D+: U$1.21, U$3.D+
- new net D-: U$1.22, U$3.D-
- new net MCLR: 10K_R3.1, PICKIT.1, RESET.3, U$1.1
- new net N$3: 330_R1.1
- new net OSC1: 8MHZRES.1, U$1.9
- new net OSC2: 8MHZRES.3, U$1.10
- new net USBID: U$1.14, U$3.ID
- new net VBUS+5: 0.1UF_1.1, J1.2, U$1.15, U$2.2, U$3.VBUS, U$4.2.PIN2, U$4.3.PIN3
- new net VDD: 0.1UF_3.1, 0.1UF_4.2, 10UF_2.1, J2.2, RED_LED.A, U$1.13, U$2.3
- net GND: now also 0.1UF_1.2, 0.1UF_3.2, 0.1UF_4.1, 10UF_2.2, 330_R2.1, J1.1, J2.1, RESET.1, U$1.8, U$3.GND, USER.1
- net N$1: now also 330_R2.2, GREEN_LED.K; no longer 8MHZRES.3, U$1.9
- net N$2: now also 330_R1.2, RED_LED.K; no longer 8MHZRES.1, U$1.10
- net N$9: now also U$1.23

Commit message: homework_2/3_commit#6
brd before error checking
Parts:
- moved 10K_R4 55.7 mm to (12.7, 41.9), turned to 270 degrees
- moved 10K_R3 49.3 mm to (17.8, 41.9), turned to 90 degrees
- moved 0.1UF_3 39.1 mm to (25.4, 2.54), turned to 180 degrees
- moved U$2 38.9 mm to (29.2, 47.0), turned to 0 degrees
- moved 0.1UF_4 22.5 mm to (35.6, 47.0), turned to 180 degrees
- moved 330_R1 17.7 mm to (10.2, 7.62), turned to 270 degrees
- moved 10UF_2 17.0 mm to (31.8, 2.54), turned to 0 degrees
- moved GREEN_LED 12.7 mm to (15.2, 11.4), turned to 180 degrees
- moved 0.1UF_1 11.5 mm to (24.1, 47.0), turned to 270 degrees
- moved 10UF_1 6.35 mm to (33.0, 24.1), turned to 90 degrees
- moved USER 5.24 mm to (7.62, 2.54), turned to 180 degrees
- moved RED_LED 4.02 mm to (15.2, 3.81), turned to 180 degrees
- moved 330_R2 2.84 mm to (7.62, 7.62), turned to 90 degrees
- moved 8MHZRES 1.27 mm to (15.2, 19.1), turned to 270 degrees
Connections:
- removed net N$3: 330_R1.1
- net GND: now also 330_R1.1
Routing:
- net VDD: track 0.00 -> 91.3 mm
- net VBUS+5: track 0.00 -> 89.4 mm, vias 0 -> 1
- net B4: track 0.00 -> 72.3 mm
- net USBID: track 0.00 -> 44.6 mm, vias 0 -> 1
- net D-: track 0.00 -> 37.7 mm, vias 0 -> 1
- net MCLR: track 0.00 -> 36.4 mm
- net D+: track 0.00 -> 35.5 mm, vias 0 -> 1
- net PGED1: track 0.00 -> 30.2 mm
- net PGEC1: track 0.00 -> 30.0 mm
- net B9: track 0.00 -> 24.9 mm
- net B8: track 0.00 -> 24.9 mm
- net B7: track 0.00 -> 24.9 mm
- net A4: track 0.00 -> 24.5 mm
- net GND: track 0.00 -> 23.2 mm, vias 0 -> 1
- net N$9: track 0.00 -> 21.7 mm
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- added copper zone on layer 16, net GND

Commit message: homework_2/3_commit#7(?)
commit after submitting final gerber
Parts:
- moved PICKIT 0.64 mm to (48.9, 48.3)
Connections:
- removed net N$8: 0.1UF_2.2, PICKIT.3, U$1.27
- net GND: now also 0.1UF_2.2, PICKIT.3, U$1.27
Routing:
- net GND: track 23.2 -> 45.3 mm
- net N$8: track 21.7 -> 0.00 mm
- net D-: track 37.7 -> 44.5 mm
- net VBUS+5: track 89.4 -> 85.2 mm
- net B3: track 21.4 -> 22.9 mm
- net B4: track 72.3 -> 71.1 mm, vias 0 -> 1
- net MCLR: track 36.4 -> 37.0 mm
- net PGEC1: track 30.0 -> 30.5 mm
Other:
- board text added: "+ -"
- board text added: "+ 10uF -"
- board text added: "++"
- board text added: "0.1uF"
- board text added: "10K"
- board text added: "330"
- board text added: ">"
- board text added: "Michael Worthington ME-433 4/14/2016"
- board text added: "reset"
- board text added: "user"
